File: Hardware Main/Electronics/Backplane/CombinedBackplane01.sch (EAGLE design)
At the start: 69 parts, among them J101 M20X2_STR_MPTH, J102 M20X2_STR_MPTH, J103 M20X2_STR_MPTH, J104 M20X2_HARFLEX_M, J105 M20X2_STR_MPTH, J106 M20X2_STR_MPTH, J107 M20X2_STR_MPTH, J108 M20X2_STR_MPTH, J109 M05X2_SMD_0.050_NOCREAM, J110 M04X2_0.050_SMD_NO_CREAM, J111 M04X2_0.050_SMD_NO_CREAM, J201 M20X2_STR_MPTH, J202 M20X2_STR_MPTH, J203 M20X2_STR_MPTH, J204 M20X2_HARFLEX_M, J205 M20X2_STR_MPTH, J206 M20X2_STR_MPTH, J301 M20X2_STR_MPTH, J302 M20X2_STR_MPTH, J303 M20X2_STR_MPTH, J304 M20X2_HARFLEX_M, J305 M20X2_STR_MPTH, J306 M20X2_STR_MPTH, J307 M20X2_STR_MPTH, J308 M05X2_SMD_0.050_NOCREAM, J401 M20X2_STR_MPTH, J402 M20X2_STR_MPTH, J403 M20X2_STR_MPTH, J404 M20X2_HARFLEX_M, J405 M20X2_STR_MPTH, J406 M20X2_STR_MPTH, J407 M20X2_STR_MPTH, J408 M05X2_SMD_0.050_NOCREAM, J501 M20X2_STR_MPTH, J502 M20X2_STR_MPTH, J503 M20X2_STR_MPTH, J504 M20X2_HARFLEX_M, J505 M20X2_STR_MPTH, J506 M20X2_STR_MPTH, J507 M20X2_STR_MPTH, J508 M05X2_SMD_0.050_NOCREAM, J509 M04X2_0.050_SMD_NO_CREAM, J510 M04X2_0.050_SMD_NO_CREAM

Commit message: Add .PDF of backplane schematic
Other:
- note added: "Six Layer Detector Adapter Backplane B0"
- note added: "Six Layer Detector Adapter Backplane B1"
- note added: "Six Layer Detector Adapter Backplane B2"
- note added: "Six Layer Detector Adapter Backplane B3"
- note removed: "Six Layer Detector Adapter Backplane"
Changed lines of the file:
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@@
 <grid distance="0.1" unitdist="inch" unit="inch" style="lines" multiple="1" display="no" altdistance="0.01" altunitdist="inch" altunit="inch"/>
 <layers>
-<layer number="1" name="Top" color="4" fill="1" visible="yes" active="no"/>
-<layer number="2" name="Route2" color="1" fill="3" visible="yes" active="no"/>
-<layer number="3" name="Route3" color="4" fill="3" visible="yes" active="no"/>
-<layer number="4" name="Route4" color="1" fill="4" visible="yes" active="no"/>
-<layer number="5" name="Route5" color="4" fill="4" visible="yes" active="no"/>
-<layer number="6" name="Route6" color="1" fill="8" visible="yes" active="no"/>
-<layer number="7" name="Route7" color="4" fill="8" visible="yes" active="no"/>
-<layer number="8" name="Route8" color="1" fill="2" visible="yes" active="no"/>
-<layer number="9" name="Route9" color="4" fill="2" visible="yes" active="no"/>
-<layer number="10" name="Route10" color="1" fill="7" visible="yes" active="no"/>
-<layer number="11" name="Route11" color="4" fill="7" visible="yes" active="no"/>
-<layer number="12" name="Route12" color="1" fill="5" visible="yes" active="no"/>
-<layer number="13" name="Route13" color="4" fill="5" visible="yes" active="no"/>
-<layer number="14" name="Route14" color="1" fill="6" visible="yes" active="no"/>
-<layer number="15" name="Route15" color="4" fill="6" visible="yes" active="no"/>
-<layer number="16" name="Bottom" color="1" fill="1" visible="yes" active="no"/>
-<layer number="17" name="Pads" color="2" fill="1" visible="yes" active="no"/>
-<layer number="18" name="Vias" color="2" fill="1" visible="yes" active="no"/>
-<layer number="19" name="Unrouted" color="6" fill="1" visible="yes" active="no"/>
-<layer number="20" name="Dimension" color="15" fill="1" visible="yes" active="no"/>
-<layer number="21" name="tPlace" color="7" fill="1" visible="yes" active="no"/>
-<layer number="22" name="bPlace" color="7" fill="1" visible="yes" active="no"/>
-<layer number="23" name="tOrigins" color="15" fill="1" visible="yes" active="no"/>
-<layer number="24" name="bOrigins" color="15" fill="1" visible="yes" active="no"/>
-<layer number="25" name="tNames" color="7" fill="1" visible="yes" active="no"/>
-<layer number="26" name="bNames" color="7" fill="1" visible="yes" active="no"/>
-<layer number="27" name="tValues" color="7" fill="1" visible="yes" active="no"/>
-<layer number="28" name="bValues" color="7" fill="1" visible="yes" active="no"/>
+<layer number="1" name="Top" color="4" fill="1" visible="no" active="no"/>
+<layer number="2" name="Route2" color="1" fill="3" visible="no" active="no"/>
+<layer number="3" name="Route3" color="4" fill="3" visible="no" active="no"/>
+<layer number="4" name="Route4" color="1" fill="4" visible="no" active="no"/>
+<layer number="5" name="Route5" color="4" fill="4" visible="no" active="no"/>
+<layer number="6" name="Route6" color="1" fill="8" visible="no" active="no"/>
+<layer number="7" name="Route7" color="4" fill="8" visible="no" active="no"/>
+<layer number="8" name="Route8" color="1" fill="2" visible="no" active="no"/>
+<layer number="9" name="Route9" color="4" fill="2" visible="no" active="no"/>
+<layer number="10" name="Route10" color="1" fill="7" visible="no" active="no"/>
+<layer number="11" name="Route11" color="4" fill="7" visible="no" active="no"/>
+<layer number="12" name="Route12" color="1" fill="5" visible="no" active="no"/>
+<layer number="13" name="Route13" color="4" fill="5" visible="no" active="no"/>
+<layer number="14" name="Route14" color="1" fill="6" visible="no" active="no"/>
+<layer number="15" name="Route15" color="4" fill="6" visible="no" active="no"/>
+<layer number="16" name="Bottom" color="1" fill="1" visible="no" active="no"/>
+<layer number="17" name="Pads" color="2" fill="1" visible="no" active="no"/>
+<layer number="18" name="Vias" color="2" fill="1" visible="no" active="no"/>
+<layer number="19" name="Unrouted" color="6" fill="1" visible="no" active="no"/>
+<layer number="20" name="Dimension" color="15" fill="1" visible="no" active="no"/>
+<layer number="21" name="tPlace" color="7" fill="1" visible="no" active="no"/>
+<layer number="22" name="bPlace" color="7" fill="1" visible="no" active="no"/>
+<layer number="23" name="tOrigins" color="15" fill="1" visible="no" active="no"/>
+<layer number="24" name="bOrigins" color="15" fill="1" visible="no" active="no"/>
+<layer number="25" name="tNames" color="7" fill="1" visible="no" active="no"/>
+<layer number="26" name="bNames" color="7" fill="1" visible="no" active="no"/>
+<layer number="27" name="tValues" color="7" fill="1" visible="no" active="no"/>
+<layer number="28" name="bValues" color="7" fill="1" visible="no" active="no"/>
 <layer number="29" name="tStop" color="7" fill="3" visible="no" active="no"/>
 <layer number="30" name="bStop" color="7" fill="6" visible="no" active="no"/>
@@
 <layer number="35" name="tGlue" color="7" fill="4" visible="no" active="no"/>
 <layer number="36" name="bGlue" color="7" fill="5" visible="no" active="no"/>
-<layer number="37" name="tTest" color="7" fill="1" visible="yes" active="no"/>
-<layer number="38" name="bTest" color="7" fill="1" visible="yes" active="no"/>
+<layer number="37" name="tTest" color="7" fill="1" visible="no" active="no"/>
+<layer number="38" name="bTest" color="7" fill="1" visible="no" active="no"/>
 <layer number="39" name="tKeepout" color="4" fill="11" visible="no" active="no"/>
 <layer number="40" name="bKeepout" color="1" fill="11" visible="no" active="no"/>
@@
 <layer number="44" name="Drills" color="7" fill="1" visible="no" active="no"/>
 <layer number="45" name="Holes" color="7" fill="1" visible="no" active="no"/>
-<layer number="46" name="Milling" color="3" fill="1" visible="yes" active="no"/>
-<layer number="47" name="Measures" color="7" fill="1" visible="yes" active="no"/>
-<layer number="48" name="Document" color="7" fill="1" visible="yes" active="no"/>
-<layer number="49" name="Reference" color="7" fill="1" visible="yes" active="no"/>
-<layer number="50" name="dxf" color="7" fill="1" visible="yes" active="no"/>
-<layer number="51" name="tDocu" color="7" fill="1" visible="yes" active="no"/>
-<layer number="52" name="bDocu" color="7" fill="1" visible="yes" active="no"/>
-<layer number="53" name="tGND_GNDA" color="7" fill="9" visible="yes" active="no"/>
-<layer number="54" name="bGND_GNDA" color="1" fill="9" visible="yes" active="no"/>
-<layer number="56" name="wert" color="7" fill="1" visible="yes" active="no"/>
-<layer number="57" name="tCAD" color="7" fill="1" visible="yes" active="no"/>
-<layer number="59" name="tCarbon" color="7" fill="1" visible="yes" active="no"/>
-<layer number="60" name="bCarbon" color="7" fill="1" visible="yes" active="no"/>
+<layer number="46" name="Milling" color="3" fill="1" visible="no" active="no"/>
+<layer number="47" name="Measures" color="7" fill="1" visible="no" active="no"/>
+<layer number="48" name="Document" color="7" fill="1" visible="no" active="no"/>
+<layer number="49" name="Reference" color="7" fill="1" visible="no" active="no"/>
+<layer number="50" name="dxf" color="7" fill="1" visible="no" active="no"/>
+<layer number="51" name="tDocu" color="7" fill="1" visible="no" active="no"/>
+<layer number="52" name="bDocu" color="7" fill="1" visible="no" active="no"/>
+<layer number="53" name="tGND_GNDA" color="7" fill="9" visible="no" active="no"/>
+<layer number="54" name="bGND_GNDA" color="1" fill="9" visible="no" active="no"/>
+<layer number="56" name="wert" color="7" fill="1" visible="no" active="no"/>
+<layer number="57" name="tCAD" color="7" fill="1" visible="no" active="no"/>
+<layer number="59" name="tCarbon" color="7" fill="1" visible="no" active="no"/>
+<layer number="60" name="bCarbon" color="7" fill="1" visible="no" active="no"/>
 <layer number="88" name="SimResults" color="9" fill="1" visible="yes" active="yes"/>
 <layer number="89" name="SimProbes" color="9" fill="1" visible="yes" active="yes"/>
@@
 <plain>
 <frame x1="0" y1="0" x2="419.1" y2="266.7" columns="8" rows="5" layer="97"/>
-<text x="17.78" y="243.84" size="6.4516" layer="97">Six Layer Detector Adapter Backplane</text>
+<text x="17.78" y="243.84" size="6.4516" layer="97">Six Layer Detector Adapter Backplane B0</text>
 <text x="81.28" y="193.04" size="2.54" layer="97">from Detector Adapter Board</text>
 <text x="330.2" y="193.04" size="2.54" layer="97">from Control Board</text>
@@
 <plain>
 <frame x1="0" y1="0" x2="419.1" y2="266.7" columns="8" rows="5" layer="97"/>
-<text x="17.78" y="243.84" size="6.4516" layer="97">Six Layer Detector Adapter Backplane</text>
+<text x="17.78" y="243.84" size="6.4516" layer="97">Six Layer Detector Adapter Backplane B1</text>
 <text x="81.28" y="193.04" size="2.54" layer="97">from Detector Adapter Board</text>
 <text x="330.2" y="193.04" size="2.54" layer="97">from Control Board</text>
@@
 <plain>
 <frame x1="0" y1="0" x2="419.1" y2="266.7" columns="8" rows="5" layer="97"/>
-<text x="17.78" y="243.84" size="6.4516" layer="97">Six Layer Detector Adapter Backplane</text>
+<text x="17.78" y="243.84" size="6.4516" layer="97">Six Layer Detector Adapter Backplane B2</text>
 <text x="81.28" y="193.04" size="2.54" layer="97">from Detector Adapter Board</text>
 <text x="330.2" y="193.04" size="2.54" layer="97">from Control Board</text>
@@
 <plain>
 <frame x1="0" y1="0" x2="419.1" y2="266.7" columns="8" rows="5" layer="97"/>
-<text x="17.78" y="243.84" size="6.4516" layer="97">Six Layer Detector Adapter Backplane</text>
+<text x="17.78" y="243.84" size="6.4516" layer="97">Six Layer Detector Adapter Backplane B3</text>
 <text x="81.28" y="193.04" size="2.54" layer="97">from Detector Adapter Board</text>
 <text x="330.2" y="193.04" size="2.54" layer="97">from Control Board</text>
